File: StabilizerShims.kicad_pcb (KiCad board)
At the start: 2 copper layers, 84 x 75 mm, 72 parts

Commit message: Revert "Begin work on v2 shim"
This reverts commit 69d9decf01aaa381d62e7f8bfa732ec1d34ae06c.
Parts:
- removed G*** (x48): LOGO, locallib:ai-4.8-combined
- removed the REF** at (127.0, 87.5)
- removed the REF** at (120.0, 87.5)
- removed the REF** at (106.0, 87.5)
- removed the REF** at (50.0, 87.5)
- removed the REF** at (127.0, 50.0)
- removed the REF** at (120.0, 50.0)
- removed the REF** at (113.0, 50.0)
- removed the REF** at (106.0, 50.0)
- removed the REF** at (99.0, 50.0)
- removed the REF** at (92.0, 50.0)
- removed the REF** at (85.0, 50.0)
- removed the REF** at (113.0, 87.5)
- removed the REF** at (78.0, 50.0)
- removed the REF** at (71.0, 50.0)
- removed the REF** at (64.0, 50.0)
- removed the REF** at (57.0, 50.0)
- removed the REF** at (50.0, 50.0)
- removed the REF** at (71.0, 87.5)
- removed the REF** at (57.0, 87.5)
- removed the REF** at (78.0, 87.5)
- removed the REF** at (99.0, 87.5)
- removed the REF** at (92.0, 87.5)
- removed the REF** at (85.0, 87.5)
- removed the REF** at (64.0, 87.5)
- added REF**: StabilizerShim-Holes, locallib:StabilizerShim-Holes, F.Cu at (214.5, 85.2)
- added REF**: StabilizerShim-Holes, locallib:StabilizerShim-Holes, F.Cu at (198.5, 64.5)
- added REF**: StabilizerShim-Holes, locallib:StabilizerShim-Holes, F.Cu at (198.5, 106.0)
- added REF**: StabilizerShim-Holes, locallib:StabilizerShim-Holes, F.Cu at (198.5, 126.8)
- added REF**: StabilizerShim-Holes, locallib:StabilizerShim-Holes, F.Cu at (190.5, 85.2)
- added REF**: StabilizerShim-Holes, locallib:StabilizerShim-Holes, F.Cu at (190.5, 64.5)
- added REF**: StabilizerShim-Holes, locallib:StabilizerShim-Holes, F.Cu at (190.5, 106.0)
- added REF**: StabilizerShim-Holes, locallib:StabilizerShim-Holes, F.Cu at (190.5, 126.8)
- added REF**: StabilizerShim-Holes, locallib:StabilizerShim-Holes, F.Cu at (182.5, 85.2)
- added REF**: StabilizerShim-Holes, locallib:StabilizerShim-Holes, F.Cu at (182.5, 64.5)
- added REF**: StabilizerShim-Holes, locallib:StabilizerShim-Holes, F.Cu at (182.5, 106.0)
- added REF**: StabilizerShim-Holes, locallib:StabilizerShim-Holes, F.Cu at (214.5, 64.5)
- added REF**: StabilizerShim-Holes, locallib:StabilizerShim-Holes, F.Cu at (182.5, 126.8)
- added REF**: StabilizerShim-Holes, locallib:StabilizerShim-Holes, F.Cu at (174.5, 85.2)
- added REF**: StabilizerShim-Holes, locallib:StabilizerShim-Holes, F.Cu at (174.5, 64.5)
- added REF**: StabilizerShim-Holes, locallib:StabilizerShim-Holes, F.Cu at (174.5, 106.0)
- added REF**: StabilizerShim-Holes, locallib:StabilizerShim-Holes, F.Cu at (174.5, 126.8)
- added REF**: StabilizerShim-Holes, locallib:StabilizerShim-Holes, F.Cu at (166.5, 85.2)
- added REF**: StabilizerShim-Holes, locallib:StabilizerShim-Holes, F.Cu at (166.5, 64.5)
- added REF**: StabilizerShim-Holes, locallib:StabilizerShim-Holes, F.Cu at (166.5, 106.0)
- added REF**: StabilizerShim-Holes, locallib:StabilizerShim-Holes, F.Cu at (166.5, 126.8)
- added REF**: StabilizerShim-Holes, locallib:StabilizerShim-Holes, F.Cu at (158.5, 85.2)
- added REF**: StabilizerShim-Holes, locallib:StabilizerShim-Holes, F.Cu at (214.5, 106.0)
- added REF**: StabilizerShim-Holes, locallib:StabilizerShim-Holes, F.Cu at (158.5, 64.5)
- added REF**: StabilizerShim-Holes, locallib:StabilizerShim-Holes, F.Cu at (158.5, 106.0)
- added REF**: StabilizerShim-Holes, locallib:StabilizerShim-Holes, F.Cu at (158.5, 126.8)
- added REF**: StabilizerShim-Holes, locallib:StabilizerShim-Holes, F.Cu at (150.5, 85.2)
- added REF**: StabilizerShim-Holes, locallib:StabilizerShim-Holes, F.Cu at (150.5, 64.5)
- added REF**: StabilizerShim-Holes, locallib:StabilizerShim-Holes, F.Cu at (150.5, 106.0)
- added REF**: StabilizerShim-Holes, locallib:StabilizerShim-Holes, F.Cu at (150.5, 126.8)
- added REF**: StabilizerShim-Holes, locallib:StabilizerShim-Holes, F.Cu at (142.5, 85.2)
- added REF**: StabilizerShim-Holes, locallib:StabilizerShim-Holes, F.Cu at (142.5, 64.5)
- added REF**: StabilizerShim-Holes, locallib:StabilizerShim-Holes, F.Cu at (142.5, 106.0)
- added REF**: StabilizerShim-Holes, locallib:StabilizerShim-Holes, F.Cu at (214.5, 126.8)
- added REF**: StabilizerShim-Holes, locallib:StabilizerShim-Holes, F.Cu at (142.5, 126.8)
- added REF**: StabilizerShim-Holes, locallib:StabilizerShim-Holes, F.Cu at (134.5, 85.2)
- added REF**: StabilizerShim-Holes, locallib:StabilizerShim-Holes, F.Cu at (134.5, 64.5)
- added REF**: StabilizerShim-Holes, locallib:StabilizerShim-Holes, F.Cu at (134.5, 106.0)
- added REF**: StabilizerShim-Holes, locallib:StabilizerShim-Holes, F.Cu at (134.5, 126.8)
- added REF**: StabilizerShim-Holes, locallib:StabilizerShim-Holes, F.Cu at (126.5, 64.5)
- added REF**: StabilizerShim-Holes, locallib:StabilizerShim-Holes, F.Cu at (126.5, 85.2)
- added REF**: StabilizerShim-Holes, locallib:StabilizerShim-Holes, F.Cu at (126.5, 106.0)
- added REF**: StabilizerShim-Holes, locallib:StabilizerShim-Holes, F.Cu at (126.5, 126.8)
- added REF**: StabilizerShim-Holes, locallib:StabilizerShim-Holes, F.Cu at (206.5, 85.2)
- added REF**: StabilizerShim-Holes, locallib:StabilizerShim-Holes, F.Cu at (206.5, 64.5)
- added REF**: StabilizerShim-Holes, locallib:StabilizerShim-Holes, F.Cu at (206.5, 106.0)
- added REF**: StabilizerShim-Holes, locallib:StabilizerShim-Holes, F.Cu at (206.5, 126.8)
- added REF**: StabilizerShim-Holes, locallib:StabilizerShim-Holes, F.Cu at (198.5, 85.2)
Routing:
- added copper zone on F.Cu, net (none)
Other:
- board size 84 x 75 mm -> 96 x 83 mm

Commit message: Update StabilizerShims.kicad_pcb
Parts:
- added G***: LOGO, locallib:ai-outline-7.6 - Copy, F.Cu at (214.5, 127.2)
- added G***: LOGO, locallib:ai-outline-7.6 - Copy, F.Cu at (142.5, 127.2)
- added G***: LOGO, locallib:ai-outline-7.6 - Copy, F.Cu at (134.5, 127.2)
- added G***: LOGO, locallib:ai-outline-7.6 - Copy, F.Cu at (126.5, 127.2)
- added G***: LOGO, locallib:ai-outline-7.6 - Copy, F.Cu at (214.5, 106.5)
- added G***: LOGO, locallib:ai-outline-7.6 - Copy, F.Cu at (206.5, 106.5)
- added G***: LOGO, locallib:ai-outline-7.6 - Copy, F.Cu at (198.5, 106.5)
- added G***: LOGO, locallib:ai-outline-7.6 - Copy, F.Cu at (190.5, 106.5)
- added G***: LOGO, locallib:ai-outline-7.6 - Copy, F.Cu at (182.5, 106.5)
- added G***: LOGO, locallib:ai-outline-7.6 - Copy, F.Cu at (174.5, 106.5)
- added G***: LOGO, locallib:ai-outline-7.6 - Copy, F.Cu at (166.5, 106.5)
- added G***: LOGO, locallib:ai-outline-7.6 - Copy, F.Cu at (206.5, 127.2)
- added G***: LOGO, locallib:ai-outline-7.6 - Copy, F.Cu at (158.5, 106.5)
- added G***: LOGO, locallib:ai-outline-7.6 - Copy, F.Cu at (150.5, 106.5)
- added G***: LOGO, locallib:ai-outline-7.6 - Copy, F.Cu at (142.5, 106.5)
- added G***: LOGO, locallib:ai-outline-7.6 - Copy, F.Cu at (134.5, 106.5)
- added G***: LOGO, locallib:ai-outline-7.6 - Copy, F.Cu at (126.5, 106.5)
- added G***: LOGO, locallib:ai-outline-7.6 - Copy, F.Cu at (214.5, 85.8)
- added G***: LOGO, locallib:ai-outline-7.6 - Copy, F.Cu at (206.5, 85.8)
- added G***: LOGO, locallib:ai-outline-7.6 - Copy, F.Cu at (198.5, 85.8)
- added G***: LOGO, locallib:ai-outline-7.6 - Copy, F.Cu at (190.5, 85.8)
- added G***: LOGO, locallib:ai-outline-7.6 - Copy, F.Cu at (182.5, 85.8)
- added G***: LOGO, locallib:ai-outline-7.6 - Copy, F.Cu at (198.5, 127.2)
- added G***: LOGO, locallib:ai-outline-7.6 - Copy, F.Cu at (174.5, 85.8)
- added G***: LOGO, locallib:ai-outline-7.6 - Copy, F.Cu at (166.5, 85.8)
- added G***: LOGO, locallib:ai-outline-7.6 - Copy, F.Cu at (158.5, 85.8)
- added G***: LOGO, locallib:ai-outline-7.6 - Copy, F.Cu at (150.5, 85.8)
- added G***: LOGO, locallib:ai-outline-7.6 - Copy, F.Cu at (142.5, 85.8)
- added G***: LOGO, locallib:ai-outline-7.6 - Copy, F.Cu at (134.5, 85.8)
- added G***: LOGO, locallib:ai-outline-7.6 - Copy, F.Cu at (126.5, 85.8)
- added G***: LOGO, locallib:ai-outline-7.6 - Copy, F.Cu at (214.5, 65.0)
- added G***: LOGO, locallib:ai-outline-7.6 - Copy, F.Cu at (206.5, 65.0)
- added G***: LOGO, locallib:ai-outline-7.6 - Copy, F.Cu at (198.5, 65.0)
- added G***: LOGO, locallib:ai-outline-7.6 - Copy, F.Cu at (190.5, 127.2)
- added G***: LOGO, locallib:ai-outline-7.6 - Copy, F.Cu at (190.5, 65.0)
- added G***: LOGO, locallib:ai-outline-7.6 - Copy, F.Cu at (182.5, 65.0)
- added G***: LOGO, locallib:ai-outline-7.6 - Copy, F.Cu at (174.5, 65.0)
- added G***: LOGO, locallib:ai-outline-7.6 - Copy, F.Cu at (166.5, 65.0)
- added G***: LOGO, locallib:ai-outline-7.6 - Copy, F.Cu at (158.5, 65.0)
- added G***: LOGO, locallib:ai-outline-7.6 - Copy, F.Cu at (150.5, 65.0)
- added G***: LOGO, locallib:ai-outline-7.6 - Copy, F.Cu at (142.5, 65.0)
- added G***: LOGO, locallib:ai-outline-7.6 - Copy, F.Cu at (134.5, 65.0)
- added G***: LOGO, locallib:ai-outline-7.6 - Copy, F.Cu at (126.5, 65.0)
- added G***: LOGO, locallib:ai-outline-7.6 - Copy, F.Cu at (182.5, 127.2)
- added G***: LOGO, locallib:ai-outline-7.6 - Copy, F.Cu at (174.5, 127.2)
- added G***: LOGO, locallib:ai-outline-7.6 - Copy, F.Cu at (166.5, 127.2)
- added G***: LOGO, locallib:ai-outline-7.6 - Copy, F.Cu at (158.5, 127.2)
- added G***: LOGO, locallib:ai-outline-7.6 - Copy, F.Cu at (150.5, 127.2)
Other:
- outline, holes or cut-outs redrawn
